File: business_card_v2/business_card_v2.kicad_sch (KiCad schematic)
At the start: 0 parts

Commit message: created ch32 symbols. added PCB USBC, created board outline
Parts:
- added J1: (no value), footprints:PCBTypeC_14P, symbol PCB_USBC:PCBTypeC_14P
- added M1: CH32X035F7P6, Package_SO:TSSOP-20_4.4x6.5mm_P0.65mm, symbol WCH_Library:CH32X035F7P6
- added U1, U10, U2, U3, U4, U5, U6, U7, U8, U9: CH32V006F8P6, Package_SO:TSSOP-20_4.4x6.5mm_P0.65mm, symbol WCH_Library:CH32V006F8P6

Commit message: bottom left to top right pins
Parts:
- removed U8: CH32V006F8P6, Package_SO:TSSOP-20_4.4x6.5mm_P0.65mm, symbol WCH_Library:CH32V006F8P6
- added C1, C11, C12, C13, C14, C15, C16, C17, C18, C19, C2, C20, C21, C22, C23, C26, C3, C4, C5, C6, C8, C9: 100nF, Capacitor_SMD:C_0603_1608Metric, symbol Device:C
- added C10, C7: 10uF, Capacitor_SMD:C_0603_1608Metric, symbol Device:C
- added D1, D2, D3, D4, D5, D6, D7, D8, D9: LED, LED_SMD:LED_1206_3216Metric, symbol Device:LED
- added P1: AMS1117-3.3, Package_TO_SOT_SMD:SOT-223-3_TabPin2, symbol Regulator_Linear:AMS1117-3.3
- added R10, R11, R3, R4, R5, R6, R7, R8, R9: 1k, Resistor_SMD:R_0603_1608Metric, symbol Device:R
- added R2: 10k, Resistor_SMD:R_0603_1608Metric, symbol Device:R
- added S1_GP0, S1_GP1, S1_GP10, S1_GP11, S1_GP12, S1_GP13, S1_GP2, S1_GP3, S1_GP4, S1_GP5, S1_GP6, S1_GP7, S1_GP8, S1_GP9, S2_GP0, S2_GP1, S2_GP10, S2_GP11, S2_GP12, S2_GP13, S2_GP2, S2_GP3, S2_GP4, S2_GP5, S2_GP6, S2_GP7, S2_GP8, S2_GP9, S3_GP0, S3_GP1, S3_GP10, S3_GP11, S3_GP12, S3_GP13, S3_GP2, S3_GP3, S3_GP4, S3_GP5, S3_GP6, S3_GP7, S3_GP8, S3_GP9, S4_GP0, S4_GP1, S4_GP10, S4_GP11, S4_GP12, S4_GP13, S4_GP2, S4_GP3, S4_GP4, S4_GP5, S4_GP6, S4_GP7, S4_GP8, S4_GP9, S5_GP0, S5_GP1, S5_GP10, S5_GP11, S5_GP12, S5_GP13, S5_GP2, S5_GP3, S5_GP4, S5_GP5, S5_GP6, S5_GP7, S5_GP8, S5_GP9, S6_GP0, S6_GP1, S6_GP10, S6_GP11, S6_GP12, S6_GP13, S6_GP2, S6_GP3, S6_GP4, S6_GP5, S6_GP6, S6_GP7, S6_GP8, S6_GP9, S7_GP0, S7_GP1, S7_GP10, S7_GP11, S7_GP12, S7_GP13, S7_GP2, S7_GP3, S7_GP4, S7_GP5, S7_GP6, S7_GP7, S7_GP8, S7_GP9, S8_GP0, S8_GP1, S8_GP10, S8_GP11, S8_GP12, S8_GP13, S8_GP2, S8_GP3, S8_GP4, S8_GP5, S8_GP6, S8_GP7, S8_GP8, S8_GP9, S9_GP0, S9_GP1, S9_GP10, S9_GP11, S9_GP12, S9_GP13, S9_GP2, S9_GP3, S9_GP4, S9_GP5, S9_GP6, S9_GP7, S9_GP8, S9_GP9: (no value), TestPoint:TestPoint_Pad_D1.0mm, symbol Connector:TestPoint
- added SW3: SW_Push, Button_Switch_SMD:SW_SPST_TL3342, symbol Switch:SW_Push
- added TP1: SWIO_N1, TestPoint:TestPoint_Pad_D2.0mm, symbol Connector:TestPoint
- added TP11: SWDIO_M, TestPoint:TestPoint_Pad_D2.0mm, symbol Connector:TestPoint
- added TP12: SWCLK_M, TestPoint:TestPoint_Pad_D2.0mm, symbol Connector:TestPoint
- added TP13: GND, TestPoint:TestPoint_Pad_D2.0mm, symbol Connector:TestPoint
- added TP14: BUS_MOSI, TestPoint:TestPoint_Pad_D2.0mm, symbol Connector:TestPoint
- added TP15: BUS_MISO, TestPoint:TestPoint_Pad_D2.0mm, symbol Connector:TestPoint
- added TP2: SWIO_N2, TestPoint:TestPoint_Pad_D2.0mm, symbol Connector:TestPoint
- added TP3: SWIO_N3, TestPoint:TestPoint_Pad_D2.0mm, symbol Connector:TestPoint
- added TP4: SWIO_N4, TestPoint:TestPoint_Pad_D2.0mm, symbol Connector:TestPoint
- added TP5: SWIO_N5, TestPoint:TestPoint_Pad_D2.0mm, symbol Connector:TestPoint
- added TP6: SWIO_N6, TestPoint:TestPoint_Pad_D2.0mm, symbol Connector:TestPoint
- added TP7: SWIO_N7, TestPoint:TestPoint_Pad_D2.0mm, symbol Connector:TestPoint
- added TP8: SWIO_N8, TestPoint:TestPoint_Pad_D2.0mm, symbol Connector:TestPoint
- added TP9: SWIO_N9, TestPoint:TestPoint_Pad_D2.0mm, symbol Connector:TestPoint
- renumbered U9 to U7, U10 to U8, U7 to U9
Connections:
- net at U6.1 (PD4): now also S6_GP0.1
- net at U6.10 (PC0): now also S6_GP4.1
- net at U6.11 (PC1): now also S6_GP5.1
- net at U6.12 (PC2): now also S6_GP6.1
- net at U6.13 (PC3): now also S6_GP7.1
- net at U6.14 (PC4): now also S6_GP8.1
- net at U6.15 (PC5): now also S6_GP9.1
- net at U6.16 (PC6): now also S6_GP10.1
- net at U6.17 (PC7): now also S6_GP11.1
- net SWIO_N6: now reaches U6.18 (PD1/SWIO)
- net SWIO_N6: now also TP6.1
- net at U6.19 (PD2): now also S6_GP12.1
- net BUS_MISO: now reaches U6.2 (PD5/TX)
- net BUS_MISO: now also M1.9 (PA3/RX2), U1.2 (PD5/TX), U2.2 (PD5/TX), U3.2 (PD5/TX), U4.2 (PD5/TX), U5.2 (PD5/TX), U7.2 (PD5/TX), U8.2 (PD5/TX), U9.2 (PD5/TX), TP15.1
- net at U6.20 (PD3): now also R8.1, S6_GP13.1
- net BUS_MOSI: now reaches U6.3 (PD6/RX)
- net BUS_MOSI: now also M1.8 (PA2/TX2), U1.3 (PD6/RX), U2.3 (PD6/RX), U3.3 (PD6/RX), U4.3 (PD6/RX), U5.3 (PD6/RX), U7.3 (PD6/RX), U8.3 (PD6/RX), U9.3 (PD6/RX), TP14.1
- net NRST_S6: now reaches U6.4 (PD7/RST)
- net NRST_S6: now also M1.11 (PA5), C16.1
- net at U6.5 (PA1): now also S6_GP1.1
- net at U6.6 (PA2): now also S6_GP2.1
- net GND: now reaches U6.7 (VSS)
- net GND: now also J1.A1 (GND), J1.A12 (GND), J1.B1 (GND), J1.B12 (GND), M1.15 (GND), U1.7 (VSS), U2.7 (VSS), U3.7 (VSS), U4.7 (VSS), U5.7 (VSS), U7.7 (VSS), U8.7 (VSS), U9.7 (VSS), C1.2, C10.2, C11.2, C12.1, C13.2, C14.1, C15.1, C16.2, C17.1, C18.2, C19.1, C2.1, C20.2, C21.1, C22.2, C23.1, C26.2, C3.2, C4.1, C5.2, C6.1, C7.2, C8.2, C9.2, D1.1 (K), D2.1 (K), D3.1 (K), D4.1 (K), D5.1 (K), D6.1 (K), D7.1 (K), D8.1 (K), D9.1 (K), P1.1 (GND), SW3.1, TP13.1
- net at U6.8 (PD0): now also S6_GP3.1
- net +3.3V: now reaches U6.9 (VDD)
- net +3.3V: now also M1.16 (VDD), U1.9 (VDD), U2.9 (VDD), U3.9 (VDD), U4.9 (VDD), U5.9 (VDD), U7.9 (VDD), U8.9 (VDD), U9.9 (VDD), C10.1, C12.2, C14.2, C15.2, C17.2, C19.2, C2.2, C21.2, C23.2, C4.2, C6.2, C9.1, P1.2 (VO), R2.2
- net at U9.1 (PD4): now also S9_GP0.1
- net at U9.10 (PC0): now also S9_GP4.1
- net at U9.11 (PC1): now also S9_GP5.1
- net at U9.12 (PC2): now also S9_GP6.1
- net at U9.13 (PC3): now also S9_GP7.1
- net at U9.14 (PC4): now also S9_GP8.1
- net at U9.15 (PC5): now also S9_GP9.1
- net at U9.16 (PC6): now also S9_GP10.1
- net at U9.17 (PC7): now also S9_GP11.1
- net SWIO_N9: now reaches U9.18 (PD1/SWIO)
- net SWIO_N9: now also TP9.1
- net at U9.19 (PD2): now also S9_GP12.1
- net at U9.20 (PD3): now also R11.1, S9_GP13.1
- net NRST_S9: now reaches U9.4 (PD7/RST)
- net NRST_S9: now also M1.14 (PB1/RX4), C22.1
- net at U9.5 (PA1): now also S9_GP1.1
- net at U9.6 (PA2): now also S9_GP2.1
- net at U9.8 (PD0): now also S9_GP3.1
- net +5V: now reaches J1.A4 (VBUS)
- net +5V: now also J1.A9 (VBUS), J1.B4 (VBUS), J1.B9 (VBUS), C7.1, C8.1, P1.3 (VI)
- net CC1: now reaches J1.A5 (CC1)
- net CC1: now also M1.2 (PC14/CC1)
- net D+: now reaches J1.A6 (DP1)
- net D+: now also J1.B6 (DP2), M1.17 (PC16/UDM)
- net D-: now reaches J1.A7 (DN1)
- net D-: now also J1.B7 (DN2), M1.18 (PC17/UDP)
- net at U5.1 (PD4): now also S5_GP0.1
- net at U5.10 (PC0): now also S5_GP4.1
- net at U5.11 (PC1): now also S5_GP5.1
- net at U5.12 (PC2): now also S5_GP6.1
- net at U5.13 (PC3): now also S5_GP7.1
- net at U5.14 (PC4): now also S5_GP8.1
- net at U5.15 (PC5): now also S5_GP9.1
- net at U5.16 (PC6): now also S5_GP10.1
- net at U5.17 (PC7): now also S5_GP11.1
- net SWIO_N5: now reaches U5.18 (PD1/SWIO)
- net SWIO_N5: now also TP5.1
- net at U5.19 (PD2): now also S5_GP12.1
- net at U5.20 (PD3): now also R7.1, S5_GP13.1
- net NRST_S5: now reaches U5.4 (PD7/RST)
- net NRST_S5: now also M1.10 (PA4), C13.1
- net at U5.5 (PA1): now also S5_GP1.1
- net at U5.6 (PA2): now also S5_GP2.1
- net at U5.8 (PD0): now also S5_GP3.1
- net NRST_S1: now reaches M1.1 (PB12)
- net NRST_S1: now also U1.4 (PD7/RST), C1.1
- net NRST_S7: now reaches M1.12 (PA6)
- net NRST_S7: now also U7.4 (PD7/RST), C18.1
- net NRST_S8: now reaches M1.13 (PA7)
- net NRST_S8: now also U8.4 (PD7/RST), C20.1
- net SWDIO_M: now reaches M1.19 (PC18/DIO)
- net SWDIO_M: now also TP11.1
- net SWCLK_M: now reaches M1.20 (PC19/DCK)
- net SWCLK_M: now also TP12.1
- net NRST_MASTER: now reaches M1.4 (PC3/RST)
- net NRST_MASTER: now also C26.1, R2.1, SW3.2
- net NRST_S2: now reaches M1.5 (PC1)
- net NRST_S2: now also U2.4 (PD7/RST), C3.1
- net NRST_S3: now reaches M1.6 (PA0)
- net NRST_S3: now also U3.4 (PD7/RST), C5.1
- net NRST_S4: now reaches M1.7 (PA1)
- net NRST_S4: now also U4.4 (PD7/RST), C11.1
- net at U1.1 (PD4): now also S1_GP0.1
- net at U1.10 (PC0): now also S1_GP4.1
- net at U1.11 (PC1): now also S1_GP5.1
- net at U1.12 (PC2): now also S1_GP6.1
- net at U1.13 (PC3): now also S1_GP7.1
- net at U1.14 (PC4): now also S1_GP8.1
- net at U1.15 (PC5): now also S1_GP9.1
- net at U1.16 (PC6): now also S1_GP10.1
- net at U1.17 (PC7): now also S1_GP11.1
- net SWIO_N1: now reaches U1.18 (PD1/SWIO)
- net SWIO_N1: now also TP1.1
- net at U1.19 (PD2): now also S1_GP12.1
- net at U1.20 (PD3): now also R3.1, S1_GP13.1
- net at U1.5 (PA1): now also S1_GP1.1
- net at U1.6 (PA2): now also S1_GP2.1
- net at U1.8 (PD0): now also S1_GP3.1
- net at U7.1 (PD4): now also S7_GP0.1
- net at U7.10 (PC0): now also S7_GP4.1
- net at U7.11 (PC1): now also S7_GP5.1
- net at U7.12 (PC2): now also S7_GP6.1
- net at U7.13 (PC3): now also S7_GP7.1
- net at U7.14 (PC4): now also S7_GP8.1
- net at U7.15 (PC5): now also S7_GP9.1
- net at U7.16 (PC6): now also S7_GP10.1
- net at U7.17 (PC7): now also S7_GP11.1
- net SWIO_N7: now reaches U7.18 (PD1/SWIO)
- net SWIO_N7: now also TP7.1
- net at U7.19 (PD2): now also S7_GP12.1
- net at U7.20 (PD3): now also R9.1, S7_GP13.1
- net at U7.5 (PA1): now also S7_GP1.1
- net at U7.6 (PA2): now also S7_GP2.1
- net at U7.8 (PD0): now also S7_GP3.1
- net at U2.1 (PD4): now also S2_GP0.1
- net at U2.10 (PC0): now also S2_GP4.1
- net at U2.11 (PC1): now also S2_GP5.1
- net at U2.12 (PC2): now also S2_GP6.1
- net at U2.13 (PC3): now also S2_GP7.1
- net at U2.14 (PC4): now also S2_GP8.1
- net at U2.15 (PC5): now also S2_GP9.1
- net at U2.16 (PC6): now also S2_GP10.1
- net at U2.17 (PC7): now also S2_GP11.1
- net SWIO_N2: now reaches U2.18 (PD1/SWIO)
- net SWIO_N2: now also TP2.1
- net at U2.19 (PD2): now also S2_GP12.1
- net at U2.20 (PD3): now also R4.1, S2_GP13.1
- net at U2.5 (PA1): now also S2_GP1.1
- net at U2.6 (PA2): now also S2_GP2.1
- net at U2.8 (PD0): now also S2_GP3.1
- net at U3.1 (PD4): now also S3_GP0.1
- net at U3.10 (PC0): now also S3_GP4.1
- net at U3.11 (PC1): now also S3_GP5.1
- net at U3.12 (PC2): now also S3_GP6.1
- net at U3.13 (PC3): now also S3_GP7.1
- net at U3.14 (PC4): now also S3_GP8.1
- net at U3.15 (PC5): now also S3_GP9.1
- net at U3.16 (PC6): now also S3_GP10.1
- net at U3.17 (PC7): now also S3_GP11.1
- net SWIO_N3: now reaches U3.18 (PD1/SWIO)
- net SWIO_N3: now also TP3.1
- net at U3.19 (PD2): now also S3_GP12.1
- net at U3.20 (PD3): now also R5.1, S3_GP13.1
- net at U3.5 (PA1): now also S3_GP1.1
- net at U3.6 (PA2): now also S3_GP2.1
- net at U3.8 (PD0): now also S3_GP3.1
- net at U8.1 (PD4): now also S8_GP0.1
- net at U8.10 (PC0): now also S8_GP4.1
- net at U8.11 (PC1): now also S8_GP5.1
- net at U8.12 (PC2): now also S8_GP6.1
- net at U8.13 (PC3): now also S8_GP7.1
- net at U8.14 (PC4): now also S8_GP8.1
- net at U8.15 (PC5): now also S8_GP9.1
- net at U8.16 (PC6): now also S8_GP10.1
- net at U8.17 (PC7): now also S8_GP11.1
- net SWIO_N8: now reaches U8.18 (PD1/SWIO)
- net SWIO_N8: now also TP8.1
- net at U8.19 (PD2): now also S8_GP12.1
- net at U8.20 (PD3): now also R10.1, S8_GP13.1
- net at U8.5 (PA1): now also S8_GP1.1
- net at U8.6 (PA2): now also S8_GP2.1
- net at U8.8 (PD0): now also S8_GP3.1
- net at U4.1 (PD4): now also S4_GP0.1
- net at U4.10 (PC0): now also S4_GP4.1
- net at U4.11 (PC1): now also S4_GP5.1
- net at U4.12 (PC2): now also S4_GP6.1
- net at U4.13 (PC3): now also S4_GP7.1
- net at U4.14 (PC4): now also S4_GP8.1
- net at U4.15 (PC5): now also S4_GP9.1
- net at U4.16 (PC6): now also S4_GP10.1
- net at U4.17 (PC7): now also S4_GP11.1
- net SWIO_N4: now reaches U4.18 (PD1/SWIO)
- net SWIO_N4: now also TP4.1
- net at U4.19 (PD2): now also S4_GP12.1
- net at U4.20 (PD3): now also R6.1, S4_GP13.1
- net at U4.5 (PA1): now also S4_GP1.1
- net at U4.6 (PA2): now also S4_GP2.1
- net at U4.8 (PD0): now also S4_GP3.1
- new net: D3.2 (A), R5.2
- new net: D6.2 (A), R8.2
- new net: D7.2 (A), R9.2
- new net: D2.2 (A), R4.2
- new net: D4.2 (A), R6.2
- new net: D8.2 (A), R10.2
- new net: D9.2 (A), R11.2
- new net: D5.2 (A), R7.2
- new net: D1.2 (A), R3.2
- no-connect marks 0 -> 1
Other:
- note added: "Master MCU"
- note added: "Power (5V to 3.3V)"
- note added: "RISC-V Super Cluster (9 MCU)"
- note added: "Reset"
- note added: "Testpoints"
- note added: "USB-C"
- moved on the sheet: J1, M1, U1, U2, U3, U4, U5, U6, U7, U8, U9

Commit message: added basic traces
Parts:
- added R12, R13: 5.1k, Resistor_SMD:R_0603_1608Metric, symbol Device:R
- TP1, TP11, TP12, TP13, TP14, TP15, TP2, TP3, TP4, TP5, TP6, TP7, TP8, TP9: footprint TestPoint:TestPoint_Pad_D2.0mm -> TestPoint:TestPoint_Pad_D1.5mm
Connections:
- net +3.3V: now also R12.2, R13.2
- net BUS_MISO: now also R13.1
- net BUS_MOSI: now also R12.1

Commit message: first commit: removed 1 MCU
Parts:
- removed C22, C23: 100nF, Capacitor_SMD:C_0603_1608Metric, symbol Device:C
- removed S9_GP0, S9_GP1, S9_GP10, S9_GP11, S9_GP12, S9_GP13, S9_GP2, S9_GP3, S9_GP4, S9_GP5, S9_GP6, S9_GP7, S9_GP8, S9_GP9: (no value), TestPoint:TestPoint_Pad_D1.0mm, symbol Connector:TestPoint
- removed TP9: SWIO_N9, TestPoint:TestPoint_Pad_D1.5mm, symbol Connector:TestPoint
- removed U9: CH32V006F8P6, Package_SO:TSSOP-20_4.4x6.5mm_P0.65mm, symbol WCH_Library:CH32V006F8P6
Connections:
- net NRST_S9 is gone; now on net NRST_S8: M1.14 (PB1/RX4)
- net NRST_S6: now also M1.12 (PA6); no longer M1.11 (PA5)
- net NRST_S7: now also M1.13 (PA7); no longer M1.12 (PA6)
- net NRST_S8: no longer M1.13 (PA7)
- net at R11.1: now also M1.11 (PA5)
Other:
- note added: "RISC-V Super Cluster (8 MCU)"
- note removed: "RISC-V Super Cluster (9 MCU)"
- moved on the sheet: C1, C10, C11, C12, C13, C14, C15, C16, C17, C18, C19, C2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

Commit message: wired all GPIO
Parts:
- renumbered S1_GP4 to S1_GP0, S1_GP3 to S1_GP1, S1_GP8 to S1_GP10, S1_GP7 to S1_GP11, S1_GP6 to S1_GP12, S1_GP5 to S1_GP13, S1_GP1 to S1_GP3, S1_GP12 to S1_GP4, S1_GP13 to S1_GP5, S1_GP0 to S1_GP6, S1_GP9 to S1_GP7, S1_GP10 to S1_GP8, S1_GP11 to S1_GP9, S2_GP4 to S2_GP0, S2_GP3 to S2_GP1, S2_GP8 to S2_GP10, S2_GP7 to S2_GP11, S2_GP6 to S2_GP12, S2_GP5 to S2_GP13, S2_GP1 to S2_GP3, S2_GP12 to S2_GP4, S2_GP13 to S2_GP5, S2_GP0 to S2_GP6, S2_GP9 to S2_GP7, S2_GP10 to S2_GP8, S2_GP11 to S2_GP9, S3_GP4 to S3_GP0, S3_GP3 to S3_GP1, S3_GP8 to S3_GP10, S3_GP7 to S3_GP11, S3_GP6 to S3_GP12, S3_GP5 to S3_GP13, S3_GP1 to S3_GP3, S3_GP12 to S3_GP4, S3_GP13 to S3_GP5, S3_GP0 to S3_GP6, S3_GP9 to S3_GP7, S3_GP10 to S3_GP8, S3_GP11 to S3_GP9, S4_GP4 to S4_GP0, S4_GP3 to S4_GP1, S4_GP8 to S4_GP10, S4_GP7 to S4_GP11, S4_GP6 to S4_GP12, S4_GP5 to S4_GP13, S4_GP1 to S4_GP3, S4_GP12 to S4_GP4, S4_GP13 to S4_GP5, S4_GP0 to S4_GP6, S4_GP9 to S4_GP7, S4_GP10 to S4_GP8, S4_GP11 to S4_GP9, S5_GP4 to S5_GP0, S5_GP3 to S5_GP1, S5_GP8 to S5_GP10, S5_GP7 to S5_GP11, S5_GP6 to S5_GP12, S5_GP5 to S5_GP13, S5_GP1 to S5_GP3, S5_GP12 to S5_GP4, S5_GP13 to S5_GP5, S5_GP0 to S5_GP6, S5_GP9 to S5_GP7, S5_GP10 to S5_GP8, S5_GP11 to S5_GP9, S6_GP4 to S6_GP0, S6_GP3 to S6_GP1, S6_GP8 to S6_GP10, S6_GP7 to S6_GP11, S6_GP6 to S6_GP12, S6_GP5 to S6_GP13, S6_GP1 to S6_GP3, S6_GP12 to S6_GP4, S6_GP13 to S6_GP5, S6_GP0 to S6_GP6, S6_GP9 to S6_GP7, S6_GP10 to S6_GP8, S6_GP11 to S6_GP9, S7_GP4 to S7_GP0, S7_GP3 to S7_GP1, S7_GP8 to S7_GP10, S7_GP7 to S7_GP11, S7_GP6 to S7_GP12, S7_GP5 to S7_GP13, S7_GP1 to S7_GP3, S7_GP12 to S7_GP4, S7_GP13 to S7_GP5, S7_GP0 to S7_GP6, S7_GP9 to S7_GP7, S7_GP10 to S7_GP8, S7_GP11 to S7_GP9
Connections:
- net NRST_S1: now also M1.14 (PB1/RX4); no longer M1.1 (PB12)
- net NRST_S2: now also M1.13 (PA7); no longer M1.5 (PC1)
- net NRST_S3: now also M1.12 (PA6); no longer M1.6 (PA0)
- net NRST_S4: now also M1.10 (PA4); no longer M1.7 (PA1)
- net NRST_S5: now also M1.1 (PB12); no longer M1.10 (PA4)
- net NRST_S6: now also M1.5 (PC1); no longer M1.12 (PA6)
- net NRST_S7: now also M1.6 (PA0); no longer M1.13 (PA7)
- net NRST_S8: now also M1.7 (PA1); no longer M1.14 (PB1/RX4)
- net at S8_GP4.1: now also U8.19 (PD2); no longer U8.10 (PC0)
- net at S8_GP3.1: now also U8.5 (PA1); no longer U8.8 (PD0)
- net at S8_GP9.1: now also U8.17 (PC7); no longer U8.15 (PC5)
- net at R10.1, U8.20 (PD3): now also S8_GP5.1; no longer S8_GP13.1
- net at S8_GP8.1: now also U8.16 (PC6); no longer U8.14 (PC4)
- net at S8_GP7.1: now also U8.15 (PC5); no longer U8.13 (PC3)
- net at U8.11 (PC1): now also S8_GP13.1; no longer S8_GP5.1
- net at S8_GP12.1: now also U8.12 (PC2); no longer U8.19 (PD2)
- net at S8_GP1.1: now also U8.8 (PD0); no longer U8.5 (PA1)
- net at S8_GP0.1: now also U8.10 (PC0); no longer U8.1 (PD4)
- net at S8_GP6.1: now also U8.1 (PD4); no longer U8.12 (PC2)
- net at S8_GP11.1: now also U8.13 (PC3); no longer U8.17 (PC7)
- net at S8_GP10.1: now also U8.14 (PC4); no longer U8.16 (PC6)
Other:
- moved on the sheet: S8_GP0, S8_GP1, S8_GP10, S8_GP11, S8_GP12, S8_GP13, S8_GP3, S8_GP4, S8_GP5, S8_GP6, S8_GP7, S8_GP8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

Commit message: added reset wires and bus
Connections:
- net NRST_S1: now also M1.12 (PA6); no longer M1.14 (PB1/RX4)
- net NRST_S3: now also M1.14 (PB1/RX4); no longer M1.12 (PA6)
- net NRST_S4: now also M1.5 (PC1); no longer M1.10 (PA4)
- net NRST_S6: now also M1.6 (PA0); no longer M1.5 (PC1)
- net NRST_S7: now also M1.7 (PA1); no longer M1.6 (PA0)
- net NRST_S8: now also M1.10 (PA4); no longer M1.7 (PA1)
Changed lines of the file:
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@@
 		)
 	)
-	(label "NRST_S6"
+	(label "NRST_S4"
 		(at 469.9 200.66 180)
 		(effects
@@
 		)
 	)
-	(label "NRST_S1"
+	(label "NRST_S3"
 		(at 513.08 205.74 0)
 		(effects
@@
 		)
 	)
-	(label "NRST_S8"
+	(label "NRST_S7"
 		(at 469.9 205.74 180)
 		(effects
@@
 		)
 	)
-	(label "NRST_S3"
+	(label "NRST_S1"
 		(at 513.08 210.82 0)
 		(effects
@@
 		)
 	)
-	(label "NRST_S4"
+	(label "NRST_S8"
 		(at 469.9 213.36 180)
 		(effects
@@
 		)
 	)
-	(label "NRST_S7"
+	(label "NRST_S6"
 		(at 469.9 203.2 180)
 		(effects
